File: smbussy.kicad_pcb (KiCad board)
At the start: 2 copper layers, 28 x 28 mm, 24 parts, among them J101 USB_C_Receptacle_USB2.0, J102 MAIN_OUT, J103 SEC_OUT, U101 USBLC6-2SC6, U102 CP2112, U103 LM1117-3.3

Commit message: finish layout
Parts:
- added JP1: PU_VSEL, Jumper:SolderJumper-3_P1.3mm_Bridged12_RoundedPad1.0x1.5mm, F.Cu at (70.5, 66.2)
- added R5: 2.2k/1206, Resistor_SMD:R_0805_2012Metric_Pad1.20x1.40mm_HandSolder, F.Cu at (72.6, 62.9)
- added R6: 2.2k/1206, Resistor_SMD:R_0805_2012Metric_Pad1.20x1.40mm_HandSolder, F.Cu at (70.7, 62.9)
- moved D2 6.40 mm to (74.3, 51.6)
- moved D3 6.34 mm to (74.3, 47.3)
- moved D1 6.32 mm to (74.3, 49.5)
- moved R8 5.96 mm to (77.2, 49.0), turned to 0 degrees
- moved R1 5.76 mm to (77.2, 50.1), turned to 180 degrees
- moved R2 5.66 mm to (77.2, 51.3), turned to 180 degrees
- moved C3 0.59 mm to (74.1, 53.9), turned to 180 degrees
- moved TP1 0.09 mm to (72.3, 54.6)
- renumbered C101 to C1, C102 to C2, C103 to C3, C104 to C4, C105 to C5, D101 to D1, D102 to D2, D103 to D3, J101 to J1, J102 to J2, J103 to J3, R101 to R1, R108 to R10, R102 to R2, R103 to R3, R104 to R4, R105 to R7, R106 to R8, R107 to R9, TP101 to TP1, TP102 to TP2, U101 to U1, U102 to U2, U103 to U3
Connections:
- net Net-(D101-Pad1) renamed /LED_TX
- net Net-(D102-Pad1) renamed /LED_RX
Routing:
- net +3V3: track 16.1 -> 38.0 mm, vias 7 -> 12
- net /IO7: track 0.00 -> 15.0 mm, vias 0 -> 2
- net /IO6: track 0.00 -> 13.3 mm, vias 0 -> 2
- net /LED_TX: track 21.8 -> 11.8 mm
- net /LED_RX: track 18.9 -> 9.27 mm
- net GND: track 40.1 -> 34.5 mm
- net Net-(JP1-Pad2): track 0.00 -> 4.21 mm
- net /SCL: track 7.65 -> 11.4 mm, vias 1 -> 3
- net /SDA: track 9.90 -> 12.9 mm
- net /IO2: track 27.6 -> 25.2 mm
- net Net-(D3-Pad2): track 0.00 -> 2.36 mm
- net VBUS: track 52.8 -> 54.7 mm
- net Net-(D1-Pad2): track 0.00 -> 1.85 mm
- net Net-(D2-Pad2): track 0.00 -> 1.73 mm
- net /IO3: track 25.2 -> 23.9 mm
Other:
- board text added: "github.com/cr1tbit/smbussy"
- board text added: "pullup select"
- board text removed: "DTR"
- board text removed: "RTS"
- board text removed: "RXD"
- board text removed: "TXD"
- board text removed: "VDD"
- board text removed: "github.com/cr1tbit/lichtenprog"
