File: smbussy.kicad_sch (KiCad schematic)
At the start: 24 parts, among them J101 USB_C_Receptacle_USB2.0, J102 MAIN_OUT, J103 SEC_OUT, U101 USBLC6-2SC6, U102 CP2112, U103 LM1117-3.3

Commit message: finish layout
Parts:
- added JP1: PU_VSEL, Jumper:SolderJumper-3_P1.3mm_Bridged12_RoundedPad1.0x1.5mm, symbol Jumper:SolderJumper_3_Bridged12
- added R5, R6: 2.2k/0603, Resistor_SMD:R_0603_1608Metric_Pad0.98x0.95mm_HandSolder, symbol Device:R
- renumbered C101 to C1, C102 to C2, C103 to C3, C104 to C4, C105 to C5, D101 to D1, D102 to D2, D103 to D3, J101 to J1, J102 to J2, J103 to J3, R101 to R1, R108 to R10, R102 to R2, R103 to R3, R104 to R4, R105 to R7, R106 to R8, R107 to R9, TP101 to TP1, TP102 to TP2, U101 to U1, U102 to U2, U103 to U3
Connections:
- net +3V3: now also JP1.1 (A)
- net SCL: now also R6.2
- net SDA: now also R5.2
- net VBUS: now also JP1.3 (B)
- net LED_TX: now reaches D1.1 (K), U2.23 (GPIO.0)
- net LED_RX: now reaches D2.1 (K), U2.22 (GPIO.1)
- new net: JP1.2 (C), R5.1, R6.1
